Commit message: Description: Correction of axis and displays in RVIZ

File: elegoo_car_v3_description/urdf/elegoo_car_v3_description.urdf (robot description, URDF)
Before this commit: robot elegoo_car_v3_description, 35 links, 34 joints
Joints:
- joint motor_to_shaft_2: axis 0 -1 0 -> 0 1 0
- joint motor_to_shaft_3: axis 0 -1 0 -> 0 1 0
