Commit message: Description & Gazebo: Implemented xacro properties and materials for simulation

File: elegoo_car_v3_description/urdf/elegoo_car_v3_description.urdf.xacro (robot description, xacro)
@@ -2,4 +2,6 @@
 <robot name="elegoo_car_v3_description" xmlns:xacro="http://ros.org/wiki/xacro">
 <!--____________________XACRO PROPERTIES___________________-->
+<xacro:include filename="$(find elegoo_car_v3_description)/urdf/colors_and_materials.xacro"/>
+<xacro:include filename="$(find elegoo_car_v3_description)/urdf/elegoo_car_v3_gazebo.urdf.xacro"/>
 <!-- __________________ BASE LINK DEFINITION______________-->
     <link
@@ -27,9 +29,5 @@
             filename="package://elegoo_car_v3_description/meshes/base_link.STL" />
         </geometry>
-        <material
-            name="">
-            <color
-            rgba="0.1254 0.1254 0.1254 0.9" />
-        </material>
+        <material name="black_acrilic"/>
         </visual>
         <collision>
@@ -73,9 +71,5 @@
                 filename="package://elegoo_car_v3_description/meshes/support_${num}.STL" />
             </geometry>
-            <material
-                name="">
-                <color
-                rgba="0.6274 0.6274 0.6274 1" />
-            </material>
+            <material name="gray_metal"/>
             </visual>
             <collision>
@@ -126,9 +120,5 @@
                 filename="package://elegoo_car_v3_description/meshes/motor_${num}.STL" />
             </geometry>
-            <material
-                name="">
-                <color
-                rgba="1 1 0 1" />
-            </material>
+            <material name="yellow"/>
             </visual>
             <collision>
@@ -180,9 +170,5 @@
                 filename="package://elegoo_car_v3_description/meshes/shaft_${num}.STL" />
             </geometry>
-                <material
-                    name="">
-                    <color
-                    rgba="1 1 1 1" />
-                </material>
+                <material name="white"/>
             </visual>
             <collision>
@@ -237,9 +223,5 @@
                 filename="package://elegoo_car_v3_description/meshes/ring_${num}.STL" />
             </geometry>
-            <material
-                name="">
-                <color
-                rgba="1 1 0 1" />
-            </material>
+            <material name="yellow"/>
             </visual>
             <collision>
@@ -294,9 +276,5 @@
                 filename="package://elegoo_car_v3_description/meshes/neumatic_${num}.STL" />
             </geometry>
-            <material
-                name="">
-                <color
-                rgba="0 0 0 1" />
-            </material>
+            <material name="black"/>
             </visual>
             <collision>
@@ -323,4 +301,13 @@
             xyz="0 0 0" />
         </joint>
+      <transmission name="motor_to_shaft_${num}_transmission">
+        <type>transmission_interface/SimpleTransmission</type>
+        <joint name="motor_to_shaft_${num}">
+            <hardwareInterface>VelocityJointInterface</hardwareInterface>
+        </joint>
+        <actuator name="motor_to_shaft_${num}_motor">
+            <mechanicalReduction>1</mechanicalReduction>
+        </actuator>
+      </transmission>
     </xacro:macro>
     <xacro:macro name="hex_supports" params="num x y z">
@@ -349,9 +336,5 @@
                 filename="package://elegoo_car_v3_description/meshes/hex_support_${num}.STL" />
             </geometry>
-            <material
-                name="">
-                <color
-                rgba="0.6 0.6 0 1" />
-            </material>
+            <material name="gold"/>
             </visual>
             <collision>
@@ -379,5 +362,5 @@
     </joint>
     </xacro:macro>
-    <!-- _________________ MODEL DEFINITIONS _______________-->
+<!-- _________________ MODEL DEFINITIONS _______________-->
     <xacro:wheel_structure num="1" front="1" dir="1"/>
     <xacro:wheel_structure num="2" front="-1" dir="1"/>
@@ -390,5 +373,5 @@
     <xacro:hex_supports num="5" x="2.0042E-08" y="-0.05605" z="0.04085" />
     <xacro:hex_supports num="6" x="0.08395" y="-0.05315" z="0.04085" />
-    <!-- _________________ PLAIN DEFINITIONS _________________-->
+<!-- _________________ PLAIN DEFINITIONS _________________-->
     <link
     name="medium_plate">
@@ -415,9 +398,5 @@
           filename="package://elegoo_car_v3_description/meshes/medium_plate.STL" />
       </geometry>
-      <material
-        name="">
-        <color
-          rgba="0.1254 0.1254 0.1254 1" />
-      </material>
+      <material name="black_acrilic"/>
     </visual>
     <collision>
@@ -468,9 +447,5 @@
           filename="package://elegoo_car_v3_description/meshes/batery.STL" />
       </geometry>
-      <material
-        name="">
-        <color
-          rgba="1 1 1 1" />
-      </material>
+      <material name="black"/>
     </visual>
     <collision>
@@ -521,9 +496,5 @@
           filename="package://elegoo_car_v3_description/meshes/arduino.STL" />
       </geometry>
-      <material
-        name="">
-        <color
-          rgba="0.529411764705882 0.549019607843137 0.549019607843137 1" />
-      </material>
+      <material name="gray_base"/>
     </visual>
     <collision>
@@ -574,9 +545,5 @@
           filename="package://elegoo_car_v3_description/meshes/servo_base.STL" />
       </geometry>
-      <material
-        name="">
-        <color
-          rgba="0.1254 0.1254 0.1254 1" />
-      </material>
+      <material name="black_acrilic"/>
     </visual>
     <collision>
@@ -627,9 +594,5 @@
           filename="package://elegoo_car_v3_description/meshes/servo.STL" />
       </geometry>
-      <material
-        name="">
-        <color
-          rgba="0.2 0.2 1 0.9" />
-      </material>
+      <material name="blue_servo"/>
     </visual>
     <collision>
@@ -680,9 +643,5 @@
           filename="package://elegoo_car_v3_description/meshes/servo_shaft.STL" />
       </geometry>
-      <material
-        name="">
-        <color
-          rgba="0.1254 0.1254 0.1254 1" />
-      </material>
+      <material name="black_acrilic"/>
     </visual>
     <collision>
@@ -738,9 +697,5 @@
           filename="package://elegoo_car_v3_description/meshes/ultrasonic_support.STL" />
       </geometry>
-      <material
-        name="">
-        <color
-          rgba="0.1254 0.1254 0.1254 1" />
-      </material>
+      <material name="black_acrilic"/>
     </visual>
     <collision>
@@ -791,9 +746,5 @@
           filename="package://elegoo_car_v3_description/meshes/ultrasonic_sensor.STL" />
       </geometry>
-      <material
-        name="">
-        <color
-          rgba="0.2 0.2 1 1" />
-      </material>
+      <material name="blue_ultrasonic"/>
     </visual>
     <collision>
@@ -820,3 +771,12 @@
       xyz="0 0 0" />
   </joint>
+  <transmission name="servo_to_shaft_transmission">
+    <type>transmission_interface/SimpleTransmission</type>
+    <joint name="servo_to_shaft">
+        <hardwareInterface>VelocityJointInterface</hardwareInterface>
+    </joint>
+    <actuator name="servo_to_shaft_motor">
+        <mechanicalReduction>1</mechanicalReduction>
+    </actuator>
+  </transmission>
 </robot>
